File: imp_measure.kicad_sch (KiCad schematic)
At the start: 71 parts, among them IC1 DAC80501ZDGST, IC2 MAX660MX_NOPB, IC4 MC33202DR2G, J1 Conn_01x04_Pin, J2 USB_B_Micro, J3 Conn_01x10_Pin, J4 Conn_01x06_Pin, J5 Conn_01x10_Pin, J6 Conn_01x03_Pin, SW1 SW_SPDT, U1 AMS1117-3.3, U2 STM32F401RCT6, Y1 Crystal

Commit message: Forrasztáshoz
Parts:
- added J7: Conn_01x10_Pin, Connector_PinSocket_2.54mm:PinSocket_1x10_P2.54mm_Vertical, symbol Connector:Conn_01x10_Pin
- added J8: Conn_01x03_Pin, Connector_PinHeader_2.54mm:PinHeader_1x03_P2.54mm_Vertical, symbol Connector:Conn_01x03_Pin
Connections:
- net +3.3V_F: now also J7.10 (Pin_10)
- net ADC1_IN4_SIGNAL: now also J7.4 (Pin_4)
- net ADC1_IN5: now also J7.8 (Pin_8), J8.2 (Pin_2)
- net DAC_OUT: now also J7.9 (Pin_9), J8.1 (Pin_1)
- net DAC_OUT_FILTERED: now also J7.7 (Pin_7), J8.3 (Pin_3)
- net GND: now also J7.1 (Pin_1)
- net IMP1: now also J7.6 (Pin_6)
- net IMP2: now also J7.5 (Pin_5)
- net IMP3: now also J7.2 (Pin_2)
- net IMP4: now also J7.3 (Pin_3)
Other:
- note added: "C35 should be eliminated to keep the DAC out DC level"
